Commit message: fixed SLAM failed bug and add updata map

File: rover_description/urdf/rover.xacro (robot description, xacro)
@@ -90,5 +90,5 @@
     <child link="L_B_Wheel_link"/>
     <origin xyz="-0.18 0.125 0.05" rpy="1.570796 0 0" />
-    <axis xyz="0 0 1" />
+    <axis xyz="0 0 -1" />
     <limit effort="100" velocity="100"/>
     <!-- velocity: m/s for prismatic, rad/s for revolute -->
@@ -122,5 +122,5 @@
     <child link="R_B_Wheel_link"/>
     <origin xyz="-0.18 -0.125 0.05" rpy="1.570796 0 0" />
-    <axis xyz="0 0 1" />
+    <axis xyz="0 0 -1" />
     <limit effort="100" velocity="100"/>
     <!-- velocity: m/s for prismatic, rad/s for revolute -->
@@ -154,5 +154,5 @@
     <child link="R_F_Wheel_link"/>
     <origin xyz="0.18 -0.125 0.05" rpy="1.570796 0 0" />
-    <axis xyz="0 0 1" />
+    <axis xyz="0 0 -1" />
     <limit effort="100" velocity="100"/>
     <!-- velocity: m/s for prismatic, rad/s for revolute -->
@@ -186,5 +186,5 @@
     <child link="L_F_Wheel_link"/>
     <origin xyz="0.18 0.125 0.05" rpy="1.570796 0 0" />
-    <axis xyz="0 0 1" />
+    <axis xyz="0 0 -1" />
     <limit effort="100" velocity="100"/>
     <!-- velocity: m/s for prismatic, rad/s for revolute -->
@@ -217,5 +217,8 @@
     <parent link="base_link"/>
     <child link="hokuyo_link"/>
+    <!--
     <origin xyz="0.175 0.05 0.15" rpy="0 0 0"/>
+    -->
+    <origin xyz="0.175 0 0.19" rpy="0 0 0"/>
     <axis xyz="0 1 0" />
   </joint>
